File: Li-ion-charger.kicad_pcb (KiCad board)
At the start: 2 copper layers, 75 x 100 mm, 126 parts, among them J1 TYPE-C-31-M-12, J2 SYS_CONN(JST S2P-VH), J3 BATT_CONN(JST S2P-VH), J4 Thermistor_CONN, J5 Conn_01x04, J6 UART_CONN, Q1 AONR21307, U1 ESP32-C3-WROOM-02, U2 BQ25895RTW, U3 TPS61023DRL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

Commit message: Improve filtering
Parts:
- removed C12, C13: 10uF, No_silkscreen:C_0805_2012Metric
- removed C14: 2.2uF, No_silkscreen:C_0805_2012Metric
- removed C7: 1uF, No_silkscreen:C_0805_2012Metric
- removed kibuzzard-69087EA2: G***, kibuzzard-69087EA2
- added C39: 100nF, No_silkscreen:C_0402_1005Metric, F.Cu at (148.1, 124.4)
- added C41: 100n, No_silkscreen:C_0402_1005Metric, F.Cu at (117.6, 120.2)
- added C43: 22uF, No_silkscreen:C_0805_2012Metric, F.Cu at (118.2, 118.7)
- added C45: 22uF, No_silkscreen:C_0805_2012Metric, F.Cu at (135.7, 122.8)
- added C46: 22uF, No_silkscreen:C_0805_2012Metric, F.Cu at (137.8, 122.8)
- added C47: 22uF, No_silkscreen:C_0805_2012Metric, F.Cu at (140.1, 122.8)
- added C48: 100nF, No_silkscreen:C_0402_1005Metric, F.Cu at (141.6, 123.3)
- added C49: 22uF, No_silkscreen:C_0805_2012Metric, F.Cu at (149.4, 129.4)
- added C50: 22uF, No_silkscreen:C_0805_2012Metric, F.Cu at (149.4, 127.2)
- added C51: 22uF, No_silkscreen:C_0805_2012Metric, F.Cu at (142.2, 119.0)
- added kibuzzard-6914ED2A: G***, kibuzzard-6914ED2A, F.Cu at (138.4, 125.5)
- C10, C9: value 10uF -> 22uF
- C11: footprint No_silkscreen:C_0603_1608Metric -> No_silkscreen:C_0805_2012Metric
- C15, C16: value 10uF -> 22uF; footprint No_silkscreen:C_0603_1608Metric -> No_silkscreen:C_0805_2012Metric
- C24: footprint No_silkscreen:C_0402_1005Metric -> No_silkscreen:C_0805_2012Metric
- C5: footprint No_silkscreen:C_0805_2012Metric -> No_silkscreen:C_0603_1608Metric
- L1: footprint Inductor_SMD:L_Vishay_IHLP-2525 -> SPM6530T-2R2M:SPM6530
- R17: value 110R -> 120R; footprint No_silkscreen:R_0402_1005Metric -> No_silkscreen:R_0603_1608Metric
- moved C9 2.45 mm to (152.4, 125.8), turned to -90 degrees
- moved C16 2.15 mm to (117.8, 128.1)
- moved C15 1.55 mm to (117.8, 126.0)
- moved L1 1.34 mm to (150.5, 119.8)
- moved kibuzzard-69087ACC 1.30 mm to (147.6, 131.8)
- moved C23 1.00 mm to (120.7, 72.8)
- moved C10 0.96 mm to (149.7, 123.9)
- moved R17 0.93 mm to (118.8, 65.3), turned to -90 degrees
- moved C11 0.83 mm to (144.2, 119.0)
- moved R22 0.72 mm to (118.8, 69.4)
- moved D14 0.53 mm to (118.0, 63.3)
- moved C24 0.52 mm to (119.0, 72.7)
- moved kibuzzard-69087EC1 0.50 mm to (133.6, 123.5)
Routing:
- net VDD: track 31.6 -> 18.1 mm
- net +5V: track 103.8 -> 107.3 mm
- net VCC: track 138.3 -> 134.8 mm
- net +3.3V: track 119.4 -> 116.2 mm
- net /BATT: track 33.6 -> 34.8 mm

Commit message: feat: Add schematic pdf
Parts:
- removed kibuzzard-69087CD6: G***, kibuzzard-69087CD6
- removed kibuzzard-69087D1E: G***, kibuzzard-69087D1E
- added D15: 1N5819HW-7-F, No Silkscreen:D_SOD-123, F.Cu at (151.4, 53.6)
- added D16: 1N5819HW-7-F, No Silkscreen:D_SOD-123, F.Cu at (111.3, 71.9)
- added R14: 22R, No Silkscreen:R_0402_1005Metric, F.Cu at (144.4, 66.0)
- added R18: 22R, No Silkscreen:R_0402_1005Metric, F.Cu at (144.4, 64.5)
- C1, C10, C11, C15, C16, C2, C24, C3, C4, C43, C45, C46, C47, C49, C50, C51, C9: footprint No_silkscreen:C_0805_2012Metric -> No Silkscreen:C_0805_2012Metric
- C17, C19, C5: footprint No_silkscreen:C_0603_1608Metric -> No Silkscreen:C_0603_1608Metric
- C18, C20, C21, C22, C23, C25, C26, C27, C28, C29, C30, C31, C32, C33, C34, C35, C36, C39, C41, C48, C6, C8: footprint No_silkscreen:C_0402_1005Metric -> No Silkscreen:C_0402_1005Metric
- C37, C38: value 100n -> 100nF; footprint No_silkscreen:C_0402_1005Metric -> No Silkscreen:C_0402_1005Metric
- D10, D11, D12, D13, D3, D4, D5, D6, D7, D8, D9: footprint No_silkscreen:LED_WS2812B-2020_PLCC4_2.0x2.0mm -> No Silkscreen:LED_WS2812B-2020_PLCC4_2.0x2.0mm
- J6: footprint Connector_PinHeader_2.54mm:PinHeader_1x02_P2.54mm_Vertical -> Connector_PinHeader_2.54mm:PinHeader_1x04_P2.54mm_Vertical
- R1, R2, R3: footprint No_silkscreen:R_0805_2012Metric -> No Silkscreen:R_0805_2012Metric
- R10, R15, R16, R4: footprint No_silkscreen:R_0805_2012Metric -> No Silkscreen:R_0402_1005Metric
- R11, R12, R13, R17, R19, R20, R21, R22, R23, R5, R6, R7, R8, R9: footprint No_silkscreen:R_0603_1608Metric -> No Silkscreen:R_0402_1005Metric
- moved J6 18.7 mm to (155.7, 53.6), turned to 90 degrees
- moved C17 3.37 mm to (111.4, 67.7)
- moved C37 2.81 mm to (111.7, 66.3)
- moved C38 2.81 mm to (111.7, 63.3)
- moved L3 2.81 mm to (112.2, 64.8)
- moved R4 0.61 mm to (125.5, 144.1)
- moved R16 0.55 mm to (120.5, 122.0)
- moved R21 0.39 mm to (119.0, 108.5)
- moved R23 0.33 mm to (118.8, 78.7)
- moved kibuzzard-69087ACC 0.30 mm to (147.5, 131.4)
- moved R20 0.30 mm to (118.9, 89.3)
- moved R19 0.28 mm to (118.8, 98.5)
- moved C48 0.14 mm to (141.6, 123.1)
Connections:
- C17 pad 1: /3.3V_EN -> Net-(D15-K)
- C37 pad 1: VCC -> Net-(D15-K)
- J6 pad 1: /UART_RX -> VEE
- J6 pad 2: /UART_TX -> GND
- L3 pad 1: VCC -> Net-(D15-K)
- U1 pad 13: /USB_D- -> /USBu_D-
- U1 pad 14: /USB_D+ -> /USBu_D+
Routing:
- net Net-(D15-K): track 0.00 -> 50.4 mm, vias 0 -> 2
- net /UART_RX: track 3.85 -> 27.5 mm, vias 0 -> 1
- net /UART_TX: track 3.94 -> 24.4 mm, vias 0 -> 1
- net VCC: track 134.8 -> 126.8 mm
- net VDD: track 18.1 -> 25.7 mm
- net /3.3V_EN: track 2.84 -> 6.19 mm
- net /USB_D+: track 88.1 -> 85.4 mm
- net /USB_D-: track 88.3 -> 85.6 mm
- net VEE: track 0.00 -> 2.62 mm
- net +3.3V: track 116.2 -> 118.1 mm
- net /USBu_D+: track 0.00 -> 1.72 mm
- net /USBu_D-: track 0.00 -> 1.71 mm
- net Net-(JP1-B): track 3.66 -> 4.62 mm
- net GND: vias 189 -> 164
- added copper zone on In1.Cu, net GND
- added copper zone on In2.Cu, net GND
- removed copper zone on F.Cu, net /3.3V_EN
Other:
- copper layers 2 -> 4
