File: Li-ion-charger.kicad_sch (KiCad schematic)
At the start: 104 parts, among them J1 TYPE-C-31-M-12, J2 SYS_CONN(JST S2P-VH), J3 BATT_CONN(JST S2P-VH), J4 Thermistor_CONN, J5 Conn_01x04, J6 UART_CONN, Q1 AONR21307, U1 ESP32-C3-WROOM-02, U2 BQ25895RTW, U3 TPS61023DRL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

Commit message: Improve filtering
Parts:
- removed C12, C13: 10uF, No_silkscreen:C_0805_2012Metric, symbol Device:C
- removed C14: 2.2uF, No_silkscreen:C_0805_2012Metric, symbol Device:C
- removed C7: 1uF, No_silkscreen:C_0805_2012Metric, symbol Device:C
- added C39, C48: 100nF, No_silkscreen:C_0402_1005Metric, symbol Device:C
- added C41: 100n, No_silkscreen:C_0402_1005Metric, symbol Device:C
- added C43, C45, C46, C47, C49, C50, C51: 22uF, No_silkscreen:C_0805_2012Metric, symbol Device:C
- C10, C9: value 10uF -> 22uF
- C11: footprint No_silkscreen:C_0603_1608Metric -> No_silkscreen:C_0805_2012Metric
- C15, C16: value 10uF -> 22uF; footprint No_silkscreen:C_0603_1608Metric -> No_silkscreen:C_0805_2012Metric
- C24: footprint No_silkscreen:C_0402_1005Metric -> No_silkscreen:C_0805_2012Metric
- C5: footprint No_silkscreen:C_0805_2012Metric -> No_silkscreen:C_0603_1608Metric
- L1: footprint Inductor_SMD:L_Vishay_IHLP-2525 -> SPM6530T-2R2M:SPM6530
- R17: value 110R -> 120R; footprint No_silkscreen:R_0402_1005Metric -> No_silkscreen:R_0603_1608Metric
Connections:
- net BATT: now also C49.1, C50.1
- net CHG_PMID: now also C51.1
- net GND: now also C39.2, C41.2, C43.2, C45.2, C46.2, C47.2, C48.2, C49.2, C50.2, C51.2
- net VCC: now also C39.1, C41.1, C43.1
- net VDD: now also C45.1, C46.1, C47.1, C48.1
Other:
- note added: "Output current is 1A max"
- note removed: "1uF -> GRM219R71E105KA88D 10uF -> GRM21BR71A106KE51L 4.7uF -> GRM188R61C475KAAJD 47nF -> GRM155R71E473KA88D"
- note removed: "Output current is 2A max"
- moved on the sheet: L2, R15, R16, TP2, TP3, U3

Commit message: feat: Add schematic pdf
Parts:
- removed J6: UART_CONN, Connector_PinHeader_2.54mm:PinHeader_1x02_P2.54mm_Vertical, symbol Connector_Generic:Conn_01x02
- added D15, D16: 1N5819HW-7-F, No Silkscreen:D_SOD-123, symbol Device:D_Schottky
- added J6: UART_CONN, Connector_PinHeader_2.54mm:PinHeader_1x04_P2.54mm_Vertical, symbol Connector_Generic:Conn_01x04
- added R14, R18: 22R, No Silkscreen:R_0402_1005Metric, symbol No silk screen devices:R
- C1, C10, C11, C15, C16, C2, C24, C3, C4, C43, C45, C46, C47, C49, C50, C51, C9: footprint No_silkscreen:C_0805_2012Metric -> No Silkscreen:C_0805_2012Metric
- C17, C19, C5: footprint No_silkscreen:C_0603_1608Metric -> No Silkscreen:C_0603_1608Metric
- C18, C20, C21, C22, C23, C25, C26, C27, C28, C29, C30, C31, C32, C33, C34, C35, C36, C41, C6, C8: footprint No_silkscreen:C_0402_1005Metric -> No Silkscreen:C_0402_1005Metric
- C37, C38: value 100n -> 100nF; footprint No_silkscreen:C_0402_1005Metric -> No Silkscreen:C_0402_1005Metric
- C39, C48: value 100nF -> 0.1uF/50V; footprint No_silkscreen:C_0402_1005Metric -> No Silkscreen:C_0603_1608Metric
- D10, D11, D12, D13, D3, D4, D5, D6, D7, D8, D9: footprint No_silkscreen:LED_WS2812B-2020_PLCC4_2.0x2.0mm -> No Silkscreen:LED_WS2812B-2020_PLCC4_2.0x2.0mm
- R1, R2, R3: footprint No_silkscreen:R_0805_2012Metric -> No Silkscreen:R_0805_2012Metric
- R10, R15, R16, R4: footprint No_silkscreen:R_0805_2012Metric -> No Silkscreen:R_0402_1005Metric
- R11, R12, R13, R17, R19, R20, R21, R22, R23, R5, R6, R7, R8, R9: footprint No_silkscreen:R_0603_1608Metric -> No Silkscreen:R_0402_1005Metric
Connections:
- net 3.3V_EN: no longer C17.1
- net GND: now also J6.2 (Pin_2)
- net UART_RX: now also J6.4 (Pin_4)
- net UART_TX: now also J6.3 (Pin_3)
- net USB_D+: now also R18.1; no longer U1.14 (IO19)
- net USB_D-: now also R14.1; no longer U1.13 (IO18)
- net VCC: now also D16.2 (A); no longer C37.1, L3.1
- new net: C17.1, C37.1, D15.1 (K), D16.1 (K), L3.1
- new net USBu_D+: R18.2, U1.14 (IO19)
- new net USBu_D-: R14.2, U1.13 (IO18)
- new net VEE: D15.2 (A), J6.1 (Pin_1)
Other:
- moved on the sheet: C10, C17, C37, C38, C39, C9, J4, L3
